File: ALogShield.sch (EAGLE design)
At the start: 25 parts, among them U1 DS3231MZ/V+T

Commit message: CC-BY-SA
Other:
- note added: "1/2"
- note added: "2.2.0a"
- note added: "2/2"
- note added: "Andrew Wickert Chad Sandell"
- note added: "Released under the Creative Commons Attribution Share-Alike 3.0 License http://creativecommons.org/licenses/by-sa/3.0 Design by: Andrew D. Wickert and Chad T. Sandell"
- note removed: "1/4"
- note removed: "2.0"
- note removed: "2/4"
